Commit message: images

File: clothoid_path_ws/src/path_controller/description/car_chassis.xacro (robot description, xacro)
@@ -5,12 +5,4 @@
     <!-- base link-->
     <link name="base_link">
-    </link>
-    <!-- base foot print link -->
-    <joint name="base_footprint_joint" type="fixed">
-        <parent link="base_link"/>
-        <child link="base_footprint"/>
-        <origin xyz="0 0 0" rpy="0 0 0"/>
-    </joint>
-    <link name="base_footprint">
     </link>
     <joint name="chassis_joint" type="fixed">
